Commit message: Phase 6: LiDAR scan messages working

File: src/inventory_manager/description/robot.urdf.xacro (robot description, xacro)
@@ -1,4 +1,245 @@
 <?xml version="1.0"?>
-<robot xmlns:xacro="http://www.ros.org/wiki/xacro"  name="robot">
-    <xacro:include filename="robot_core.xacro" />
+<robot xmlns:xacro="http://www.ros.org/wiki/xacro" name="robot">
+<!-- ============================================================ -->
+<!-- Materials (used for RViz display) -->
+<!-- ============================================================ -->
+<material name="grey">
+    <color rgba="0.3 0.3 0.3 1.0"/>
+</material>
+<material name="orange">
+    <color rgba="0.9 0.6 0.1 1.0"/>
+</material>
+<material name="silver">
+    <color rgba="0.8 0.8 0.8 1.0"/>
+</material>
+<!-- ============================================================ -->
+<!-- Properties:  -->
+<!-- ============================================================ -->
+<xacro:property name="chassis_length" value="0.40"/>
+<xacro:property name="chassis_width"  value="0.30"/>
+<xacro:property name="chassis_height" value="0.15"/>
+<xacro:property name="chassis_mass"   value="5.0"/>
+<xacro:property name="wheel_radius" value="0.05"/>
+<xacro:property name="wheel_width"  value="0.04"/>
+<xacro:property name="wheel_mass"   value="0.3"/>
+<xacro:property name="wheel_separation" value="0.30"/> <!-- left-right distance between wheel centers -->
+<xacro:property name="wheelbase"        value="0.30"/> <!-- front-to-back distance between axles -->
+<xacro:property name="caster_radius" value="0.025"/>
+<xacro:property name="caster_mass"   value="0.1"/>
+<xacro:property name="lidar_radius" value="0.03"/>
+<xacro:property name="lidar_height" value="0.05"/>
+<!-- ============================================================ -->
+<!-- Reusable inertia macros -->
+<!-- ============================================================ -->
+  <xacro:macro name="box_inertia" params="mass x y z">
+    <inertial>
+      <mass value="${mass}"/>
+      <inertia
+        ixx="${(mass/12.0)*(y*y+z*z)}" ixy="0.0" ixz="0.0"
+        iyy="${(mass/12.0)*(x*x+z*z)}" iyz="0.0"
+        izz="${(mass/12.0)*(x*x+y*y)}"/>
+    </inertial>
+  </xacro:macro>
+  <xacro:macro name="cylinder_inertia" params="mass r h">
+    <inertial>
+      <mass value="${mass}"/>
+      <inertia
+        ixx="${(mass/12.0)*(3*r*r+h*h)}" ixy="0.0" ixz="0.0"
+        iyy="${(mass/12.0)*(3*r*r+h*h)}" iyz="0.0"
+        izz="${(mass/2.0)*(r*r)}"/>
+    </inertial>
+  </xacro:macro>
+  <!-- Solid sphere inertia: I = (2/5) * m * r^2 for all three axes -->
+  <xacro:macro name="sphere_inertia" params="mass r">
+    <inertial>
+      <mass value="${mass}"/>
+      <inertia
+        ixx="${(2.0/5.0)*mass*r*r}" ixy="0.0" ixz="0.0"
+        iyy="${(2.0/5.0)*mass*r*r}" iyz="0.0"
+        izz="${(2.0/5.0)*mass*r*r}"/>
+    </inertial>
+  </xacro:macro>
+  <!-- ============================================================ -->
+  <!-- Base Footprint Link and Base Link-->
+  <!-- ============================================================ -->
+  <link name="base_footprint"/>
+  <joint name="base_joint" type="fixed">
+    <parent link="base_footprint"/>
+    <child link="base_link"/>
+    <origin xyz="0 0 ${wheel_radius}" rpy="0 0 0"/>
+  </joint>
+  <!-- Base Link is the chasis of the robot -->
+  <link name="base_link">
+    <visual>
+      <origin xyz="0 0 0" rpy="0 0 0"/>
+      <geometry>
+        <box size="${chassis_length} ${chassis_width} ${chassis_height}"/>
+      </geometry>
+      <material name="grey"/>
+    </visual>
+    <collision>
+      <origin xyz="0 0 0" rpy="0 0 0"/>
+      <geometry>
+        <box size="${chassis_length} ${chassis_width} ${chassis_height}"/>
+      </geometry>
+    </collision>
+    <xacro:box_inertia mass="${chassis_mass}" x="${chassis_length}" y="${chassis_width}" z="${chassis_height}"/>
+  </link>
+  <gazebo reference="base_link">
+    <material>Gazebo/Grey</material>
+  </gazebo>
+  <!-- ============================================================ -->
+  <!-- Wheel macro                                                   -->
+  <!-- Every wheel gets identical visual/collision/inertial/joint    -->
+  <!-- structure. Whether a wheel is actually "driven" is decided    -->
+  <!-- ONLY by whether its joint name is referenced by the Gazebo    -->
+  <!-- diff_drive plugin below - rear wheels get a normal continuous-->
+  <!-- joint with no plugin attached, so they spin freely under      -->
+  <!-- rolling friction as the robot moves, exactly like an unpowered-->
+  <!-- axle.                                                          -->
+  <!-- ============================================================ -->
+  <xacro:macro name="wheel" params="prefix x_pos y_pos">
+    <link name="${prefix}_wheel_link">
+      <visual>
+        <origin xyz="0 0 0" rpy="${pi/2} 0 0"/>
+        <geometry>
+          <cylinder radius="${wheel_radius}" length="${wheel_width}"/>
+        </geometry>
+        <material name="orange"/>
+      </visual>
+      <collision>
+        <origin xyz="0 0 0" rpy="${pi/2} 0 0"/>
+        <geometry>
+          <cylinder radius="${wheel_radius}" length="${wheel_width}"/>
+        </geometry>
+      </collision>
+      <xacro:cylinder_inertia mass="${wheel_mass}" r="${wheel_radius}" h="${wheel_width}"/>
+    </link>
+    <joint name="${prefix}_wheel_joint" type="continuous">
+      <parent link="base_link"/>
+      <child link="${prefix}_wheel_link"/>
+      <origin xyz="${x_pos} ${y_pos} -${wheel_radius}" rpy="0 0 0"/>
+      <axis xyz="0 1 0"/>
+      <dynamics damping="0.1" friction="0.0"/>
+    </joint>
+    <gazebo reference="${prefix}_wheel_link">
+      <material>Gazebo/Black</material>
+      <mu1>1.0</mu1>
+      <mu2>1.0</mu2>
+    </gazebo>
+  </xacro:macro>
+  <!-- FRONT wheels: these are the ones the diff_drive plugin actuates -->
+  <xacro:wheel prefix="front_left"  x_pos="${wheelbase/2}"  y_pos="${wheel_separation/2}"/>
+  <xacro:wheel prefix="front_right" x_pos="${wheelbase/2}"  y_pos="-${wheel_separation/2}"/>
+  <!-- ============================================================ -->
+  <!-- Rear caster macro                                             -->
+  <!-- A caster is modeled as a simple sphere with very low friction -->
+  <!-- and a FIXED joint (no motor, no rotation axis needed) a    -->
+  <!-- sphere's shape lets it slide/scrub in any direction under low -->
+  <!-- friction, which is what a real swivel caster does, without    -->
+  <!-- needing to model the actual swivel mechanism.                 -->
+  <!-- ============================================================ -->
+  <xacro:macro name="caster" params="prefix x_pos y_pos">
+    <link name="${prefix}_caster_link">
+      <visual>
+        <origin xyz="0 0 0" rpy="0 0 0"/>
+        <geometry>
+          <sphere radius="${caster_radius}"/>
+        </geometry>
+        <material name="silver"/>
+      </visual>
+      <collision>
+        <origin xyz="0 0 0" rpy="0 0 0"/>
+        <geometry>
+          <sphere radius="${caster_radius}"/>
+        </geometry>
+      </collision>
+      <xacro:sphere_inertia mass="${caster_mass}" r="${caster_radius}"/>
+    </link>
+    <joint name="${prefix}_caster_joint" type="fixed">
+      <parent link="base_link"/>
+      <child link="${prefix}_caster_link"/>
+      <origin xyz="${x_pos} ${y_pos} ${-(wheel_radius+caster_radius)}" rpy="0 0 0"/>
+    </joint>
+    <gazebo reference="${prefix}_caster_link">
+      <material>Gazebo/Grey</material>
+      <mu1>0.01</mu1>
+      <mu2>0.01</mu2>
+    </gazebo>
+  </xacro:macro>
+  <!-- Rear casters: replace the old rear_left/rear_right wheels -->
+  <xacro:caster prefix="rear_left"  x_pos="-${wheelbase/2}" y_pos="${wheel_separation/2}"/>
+  <xacro:caster prefix="rear_right" x_pos="-${wheelbase/2}" y_pos="-${wheel_separation/2}"/>
+  <!-- ============================================================ -->
+  <!-- Lidar Link-->
+  <!-- ============================================================ -->
+  <link name="lidar_link">
+    <visual>
+      <geometry>
+        <cylinder radius="${lidar_radius}" length="${lidar_height}"/>
+      </geometry>
+      <material name="grey"/>
+    </visual>
+    <collision>
+      <geometry>
+        <cylinder radius="${lidar_radius}" length="${lidar_height}"/>
+      </geometry>
+    </collision>
+    <xacro:cylinder_inertia mass="0.1" r="${lidar_radius}" h="${lidar_height}"/>
+  </link>
+  <joint name="lidar_joint" type="fixed">
+    <parent link="base_link"/>
+    <child link="lidar_link"/>
+    <origin xyz="0 0 ${chassis_height/2 + lidar_height/2}" rpy="0 0 0"/>
+  </joint>
+  <gazebo reference="lidar_link">
+    <sensor name="lidar" type="gpu_lidar">
+      <pose>0 0 0 0 0 0</pose>
+      <topic>scan</topic>
+      <update_rate>10</update_rate>
+      <visualize>true</visualize>
+      <always_on>true</always_on>
+      <lidar>
+        <scan>
+          <horizontal>
+            <samples>360</samples>
+            <min_angle>-3.14159</min_angle>
+            <max_angle>3.14159</max_angle>
+          </horizontal>
+        </scan>
+        <range>
+          <min>0.1</min>
+          <max>12.0</max>
+        </range>
+      </lidar>
+    </sensor>
+  </gazebo>
+  <!-- ============================================================ -->
+  <!-- Gazebo plugins (differential drive, joint state publisher)   -->
+  <!-- NOTE: both must live inside a <gazebo> wrapper, or URDF       -->
+  <!-- ignores them. The Sensors system is NOT loaded here - it's   -->
+  <!-- already loaded once at the world level (see                  -->
+  <!-- worlds/inventory_test.sdf). Loading it a second time here     -->
+  <!-- spins up a second render thread that races the world's       -->
+  <!-- render thread to initialize the same Ogre2 scene, crashing   -->
+  <!-- gz-sim server with an Ogre::ItemIdentityException as soon as  -->
+  <!-- a sensor tries to render.                                     -->
+  <!-- ============================================================ -->
+  <gazebo>
+    <plugin filename="gz-sim-diff-drive-system" name="gz::sim::systems::DiffDrive">
+      <left_joint>front_left_wheel_joint</left_joint>
+      <right_joint>front_right_wheel_joint</right_joint>
+      <wheel_separation>${wheel_separation}</wheel_separation>
+      <wheel_radius>${wheel_radius}</wheel_radius>
+      <odom_publish_frequency>30</odom_publish_frequency>
+      <topic>cmd_vel</topic>
+      <odom_topic>odom</odom_topic>
+      <frame_id>odom</frame_id>
+      <child_frame_id>base_footprint</child_frame_id>
+    </plugin>
+    <plugin filename="gz-sim-joint-state-publisher-system" name="gz::sim::systems::JointStatePublisher">
+      <joint_name>front_left_wheel_joint</joint_name>
+      <joint_name>front_right_wheel_joint</joint_name>
+    </plugin>
+  </gazebo>
 </robot>
